Commit message: 2/27/15:08

File: mastering_ros_robot_description_pkg/urdf/sensors/seven_dof_arm.xacro (robot description, xacro)
@@ -63,8 +63,4 @@
   <xacro:gripper parent="tool"/>
 -->
-<!--
-	////////////////////////////////////////////////////////////
-	////////////////////////////////////////////////////////////
--->
   <joint name="bottom_joint" type="fixed">
 	<origin xyz="0 0 0" rpy="0 0 0"/>
@@ -89,8 +85,4 @@
 	<material>Gazebo/White</material>
   </gazebo>
-<!--
-	////////////////////////////////////////////////////////////
-	////////////////////////////////////////////////////////////
--->
   <link name="base_link">
 	<visual>
@@ -111,20 +103,12 @@
 	<material>Gazebo/White</material>
   </gazebo>
-<!--
-	////////////////////////////////////////////////////////////
-	////////////////////////////////////////////////////////////
--->
   <joint name="shoulder_pan_joint" type="revolute">
 	<parent link="base_link"/>
 	<child link="shoulder_pan_link"/>
-	<origin xyz="0 0 0.05" rpy="0 ${M_PI/2} ${M_PI*0}"/>
+	<origin xyz="0 0 0.05" rpy="0 ${M_PI/2} 0"/>
 	<axis xyz="-1 0 0"/>
 	<limit effort="300" velocity="20" lower="-2.61799" upper="1.98394"/>
 	<dynamics damping="50" friction="1"/>
   </joint>
-<!--
-	////////////////////////////////////////////////////////////
-	////////////////////////////////////////////////////////////
--->
   <link name="shoulder_pan_link">
 	<visual>
@@ -146,8 +130,4 @@
 	<material>Gazebo/Red</material>
   </gazebo>
-<!--
-	////////////////////////////////////////////////////////////
-	////////////////////////////////////////////////////////////
--->
   <joint name="shoulder_pitch_joint" type="revolute">
 	<parent link="shoulder_pan_link"/>
@@ -158,8 +138,4 @@
 	<dynamics dapming="50" friction="1"/>
   </joint>
-<!--
-	////////////////////////////////////////////////////////////
-	////////////////////////////////////////////////////////////
--->
   <link name="shoulder_pitch_link">
 	<visual>
@@ -181,8 +157,4 @@
 	<material>Gazebo/White</material>
   </gazebo>
-<!--
-	////////////////////////////////////////////////////////////
-	////////////////////////////////////////////////////////////
--->
   <joint name="elbow_roll_joint" type="revolute">
 	<parent link="shoulder_pitch_link"/>
@@ -193,8 +165,4 @@
 	<dynamics damping="50" friction="1"/>
   </joint>
-<!--
-	////////////////////////////////////////////////////////////
-	////////////////////////////////////////////////////////////
--->
   <link name="elbow_roll_link">
 	<visual>
@@ -216,21 +184,12 @@
 	<material>Gazebo/Black</material>
   </gazebo>
-<!--
-	////////////////////////////////////////////////////////////
-	////////////////////////////////////////////////////////////
--->
   <joint name="elbow_pitch_joint" type="revolute">
 	<parent link="elbow_roll_link"/>
 	<child link="elbow_pitch_link"/>
-	<origin xyz="-0.035 0 0.0" rpy="0.055 ${M_PI/2} 0"/>
-	<!-- <origin xyz="-0.035 0 0.0" rpy="${M_PI} ${M_PI/2} 0"/> -->
+	<origin xyz="-0.035 0 0" rpy="0.055 ${M_PI/2} 0"/>
 	<axis xyz="1 0 0"/>
 	<limit effort="300" velocity="1" lower="-1.59534" upper="1.9328"/>
 	<dynamics damping="50" friction="1"/>
   </joint>
-<!--
-	////////////////////////////////////////////////////////////
-	////////////////////////////////////////////////////////////
--->
   <link name="elbow_pitch_link">
 	<visual>
@@ -252,23 +211,15 @@
 	<material>Gazebo/Red</material>
   </gazebo>
-<!--
-	////////////////////////////////////////////////////////////
-	////////////////////////////////////////////////////////////
--->
   <joint name="wrist_roll_joint" type="revolute">
 	<parent link="elbow_pitch_link"/>
 	<child link="wrist_roll_link"/>
-	<origin xyz="0.0 0.0081 -0.248" rpy="0 ${M_PI/2} ${M_PI}"/>
+	<origi xyz="0.0 0.0081 -0.248" rpy="0 ${M_PI/2} ${M_PI}"/>
 	<axis xyz="1 0 0"/>
 	<limit effort="300" velocity="1" lower="-2.61799" upper="2.61288"/>
 	<dynamics damping="50" friction="1"/>
   </joint>
-<!--
-	////////////////////////////////////////////////////////////
-	////////////////////////////////////////////////////////////
--->
   <link name="wrist_roll_link">
 	<visual>
-	  <origin xyz="0 0 0" rpy="0 ${M_PI/2} 0"/>
+	  <orign xyz="0 0 0" rpy="0 ${M_PI/2} 0"/>
 	  <geometry>
 		<cylinder radius="${elbow_roll_width}" length="${elbow_roll_len}"/>
@@ -287,8 +238,4 @@
 	<material>Gazebo/Black</material>
   </gazebo>
-<!--
-	////////////////////////////////////////////////////////////
-	////////////////////////////////////////////////////////////
--->
   <joint name="wrist_pitch_joint" type="revolute">
 	<parent link="wrist_roll_link"/>
@@ -299,8 +246,4 @@
 	<dynamics damping="50" friction="1"/>
   </joint>
-<!--
-	////////////////////////////////////////////////////////////
-	////////////////////////////////////////////////////////////
--->
   <link name="wrist_pitch_link">
 	<visual>
@@ -314,5 +257,5 @@
 	  <origin xyz="0 0 0.04" rpy="0 ${M_PI/2} 0"/>
 	  <geometry>
-		<box size="${wrist_pitch_len} ${wrist_pitch_width} ${wrist_pitch_height}"/>
+		<box size="{wrist_pitch_len} ${wrist_pitch_width} ${wrist_pitch_height}"/>
 	  </geometry>
 	</collision>
@@ -322,8 +265,4 @@
 	<material>Gazebo/Black</material>
   </gazebo>
-<!--
-	////////////////////////////////////////////////////////////
-	////////////////////////////////////////////////////////////
--->
   <joint name="gripper_roll_joint" type="revolute">
 	<parent link="wrist_pitch_link"/>
@@ -334,8 +273,4 @@
 	<dynamics damping="50" friction="1"/>
   </joint>
-<!--
-	////////////////////////////////////////////////////////////
-	////////////////////////////////////////////////////////////
--->
   <link name="gripper_roll_link">
 	<visual>
@@ -355,10 +290,19 @@
   </link>
   <gazebo reference="gripper_roll_link">
-	<material>Gazebo/Red</material>
-  </gazebo>
-<!--
-	////////////////////////////////////////////////////////////
-	////////////////////////////////////////////////////////////
--->
+	<visual>
+	  <origin xyz="0 0 0" rpy="0 ${M_PI/2} 0"/>
+	  <geometry>
+		<cylinder radius="${gripper_roll_width}" length="${gripper_roll_len}"/>
+	  </geometry>
+	  <material name="Red"/>
+	</visual>
+	<collision>
+	  <origin xyz="0 0 0" rpy="0 ${M_PI/2} 0"/>
+	  <geometry>
+		<cylinder radius="${gripper_roll_width}" length="${gripper_roll_len}"/>
+	  </geometry>
+	</collision>
+	<xacro:inertial_matrix mass="1"/>
+  </gazebo>
   <joint name="finger_joint1" type="prismatic">
 	<parent link="gripper_roll_link"/>
@@ -373,8 +317,4 @@
 	<dynamics damping="50" friction="1"/>
   </joint>
-<!--
-	////////////////////////////////////////////////////////////
-	////////////////////////////////////////////////////////////
--->
   <link name="gripper_finger_link1">
 	<visual>
@@ -390,8 +330,4 @@
 	<material>Gazebo/White</material>
   </gazebo>
-<!--
-	////////////////////////////////////////////////////////////
-	////////////////////////////////////////////////////////////
--->
   <joint name="finger_jiont2" type="prismatic">
 	<parent link="gripper_roll_link"/>
@@ -402,11 +338,7 @@
 	<dynamics damping="50" friction="1"/>
   </joint>
-<!--
-	////////////////////////////////////////////////////////////
-	////////////////////////////////////////////////////////////
--->
   <link name="gripper_finger_link2">
 	<visual>
-	  <origin xyz="0.04 0.03 0"/>
+	  <orign xyz="0.04 0.03 0"/>
 	  <geometry>
 		<box size="${right_gripper_len} ${right_gripper_width} ${right_gripper_height}"/>
@@ -419,8 +351,4 @@
 	<material>Gazebo/White</material>
   </gazebo>
-<!--
-	////////////////////////////////////////////////////////////
-	////////////////////////////////////////////////////////////
--->
   <link name="grasping_frame">
 	<iertial>
@@ -438,8 +366,4 @@
 	</visual>
   </link>
-<!--
-	////////////////////////////////////////////////////////////
-	////////////////////////////////////////////////////////////
--->
   <joint name="grasping_frame_joint" type="fixed">
 	<parent link="gripper_roll_link"/>
