Commit message: updated chapter2

File: chapter2_codes/mastering_ros_robot_description_pkg/urdf/diff_wheeled_robot.xacro (robot description, xacro)
@@ -17,35 +17,35 @@
   <!-- PROPERTY LIST -->
   <!--All units in m-kg-s-radians unit system -->
-  <property name="M_PI" value="3.1415926535897931" />
-  <property name="M_PI_2" value="1.570796327" />
-  <property name="DEG_TO_RAD" value="0.017453293" />
+  <xacro:property name="M_PI" value="3.1415926535897931" />
+  <xacro:property name="M_PI_2" value="1.570796327" />
+  <xacro:property name="DEG_TO_RAD" value="0.017453293" />
   <!-- Main body radius and height -->
   <!-- Main Body Cylinder base   -->
-  <property name="base_height" value="0.02" />
-  <property name="base_radius" value="0.15" />
-  <property name="base_mass" value="5" /> <!-- in kg-->
+  <xacro:property name="base_height" value="0.02" />
+  <xacro:property name="base_radius" value="0.15" />
+  <xacro:property name="base_mass" value="5" /> <!-- in kg-->
   <!-- caster wheel radius and height -->
   <!-- caster wheel mass -->
-  <property name="caster_f_height" value="0.04" />
-  <property name="caster_f_radius" value="0.025" />
-  <property name="caster_f_mass" value="0.5" /> <!-- in kg-->
+  <xacro:property name="caster_f_height" value="0.04" />
+  <xacro:property name="caster_f_radius" value="0.025" />
+  <xacro:property name="caster_f_mass" value="0.5" /> <!-- in kg-->
   <!-- caster wheel radius and height -->
   <!-- caster wheel mass -->
-  <property name="caster_b_height" value="0.04" />
-  <property name="caster_b_radius" value="0.025" />
-  <property name="caster_b_mass" value="0.5" /> <!-- in kg-->
+  <xacro:property name="caster_b_height" value="0.04" />
+  <xacro:property name="caster_b_radius" value="0.025" />
+  <xacro:property name="caster_b_mass" value="0.5" /> <!-- in kg-->
   <!-- Wheels -->
-  <property name="wheel_mass" value="2.5" /> --> <!-- in kg-->
-  <property name="base_x_origin_to_wheel_origin" value="0.25" />
-  <property name="base_y_origin_to_wheel_origin" value="0.3" />
-  <property name="base_z_origin_to_wheel_origin" value="0.0" />
+  <xacro:property name="wheel_mass" value="2.5" /> --> <!-- in kg-->
+  <xacro:property name="base_x_origin_to_wheel_origin" value="0.25" />
+  <xacro:property name="base_y_origin_to_wheel_origin" value="0.3" />
+  <xacro:property name="base_z_origin_to_wheel_origin" value="0.0" />
   <!-- Hokuyo Laser scanner -->
-  <property name="hokuyo_size" value="0.05" />
+  <xacro:property name="hokuyo_size" value="0.05" />
   <!-- Macro for calculating inertia of cylinder -->
-  <macro name="cylinder_inertia" params="m r h">
+  <xacro:macro name="cylinder_inertia" params="m r h">
     <inertia  ixx="${m*(3*r*r+h*h)/12}" ixy = "0" ixz = "0"
               iyy="${m*(3*r*r+h*h)/12}" iyz = "0"
               izz="${m*r*r/2}" />
-  </macro>
+  </xacro:macro>
   <!-- BASE-FOOTPRINT -->
   <!-- base_footprint is a fictitious link(frame) that is on the ground right below base_link origin -->

File: chapter2_codes/mastering_ros_robot_description_pkg/urdf/pan_tilt.urdf (robot description, URDF)
Before this commit: robot pan_tilt, 3 links, 2 joints
Links:
- link base_link: mass None -> 1
- link pan_link: mass None -> 1
- link tilt_link: mass None -> 1

File: chapter2_codes/mastering_ros_robot_description_pkg/urdf/pan_tilt.xacro (robot description, xacro)
@@ -1,91 +1,90 @@
 <?xml version="1.0"?>
-<robot xmlns:xacro="https://www.ros.org/wiki/xacro"
-	   xmlns:sensor="http://playerstage.sourceforge.net/gazebo/xmlschema/#sensor"
-	   xmlns:controller="http://playerstage.sourceforge.net/gazebo/xmlschema/#controller"
-	   xmlns:interface="http://playerstage.sourceforge.net/gazebo/xmlschema/#interface"
-	   name="pan_tilt">
-  <xacro:property name="base_link_length" value="0.1"/>
-  <xacro:property name="base_link_radius" value="0.2"/>
-  <xacro:property name="pan_link_length" value="0.4"/>
-  <xacro:property name="pan_link_radius" value="0.04"/>
-  <xacro:property name="tilt_link_length" value="0.4"/>
-  <xacro:property name="tilt_link_radius" value="0.04"/>
-  <xacro:macro name="inertial_matrix" params="mass">
-	<inertial>
-	  <mass value="${mass}"/>
-	  <inertia ixx="0.5" ixy="0.0" ixz="0.0"
-				iyy="0.5" iyz="0.0"
-				izz="0.5"/>
-	</inertial>
-  </xacro:macro>
+<robot xmlns:xacro="http://www.ros.org/wiki/xacro"
+ 	xmlns:sensor="http://playerstage.sourceforge.net/gazebo/xmlschema/#sensor"
+    	xmlns:controller="http://playerstage.sourceforge.net/gazebo/xmlschema/#controller"
+    	xmlns:interface="http://playerstage.sourceforge.net/gazebo/xmlschema/#interface"
+	name="pan_tilt">
+	<xacro:property name="base_link_length" value="0.01" />
+	<xacro:property name="base_link_radius" value="0.2" />
+	<xacro:property name="pan_link_length" value="0.4" />
+	<xacro:property name="pan_link_radius" value="0.04" />
+	<xacro:property name="tilt_link_length" value="0.4" />
+	<xacro:property name="tilt_link_radius" value="0.04" />
+	<xacro:macro name="inertial_matrix" params="mass">
+               <inertial>
+                       <mass value="${mass}" />
+                       <inertia ixx="0.5" ixy="0.0" ixz="0.0"
+                                iyy="0.5" iyz="0.0"
+                                izz="0.5" />
+               </inertial>
+	</xacro:macro>
   <link name="base_link">
-	<visual>
-	  <geometry>
-		<cylinder length="${base_link_length}" radius="${base_link_radius}"/>
-	  </geometry>
-	  <origin rpy="0 0 0" xyz="0 0 0"/>
-	  <material name="yellow">
-		<color rgba="1 1 0 1"/>
-	  </material>
-	</visual>
-	<collision>
-	  <geometry>
-		<cylinder length="${base_link_length+0.02}" radius="0.2"/>
-	  </geometry>
-	  <origin rpy="0 0 0" xyz="0 0 0"/>
-	</collision>
-	  <xacro:inertial_matrix mass="1"/>
+    <visual>
+      <geometry>
+	<cylinder length="${base_link_length}" radius="${base_link_radius}"/>
+      </geometry>
+      <origin rpy="0 0 0" xyz="0 0 0"/>
+      <material name="yellow">
+        <color rgba="1 1 0 1"/>
+      </material>
+    </visual>
+    <collision>
+      <geometry>
+	<cylinder length="${base_link_length+0.02}" radius="0.2"/>
+      </geometry>
+      <origin rpy="0 0 0" xyz="0 0 0"/>
+    </collision>
+	<xacro:inertial_matrix mass="1"/>
   </link>
   <joint name="pan_joint" type="revolute">
-	<parent link="base_link"/>
-	<child link="pan_link"/>
-	<origin xyz="0 0 0.1"/>
-	<axis xyz="0 0 1"/>
-	<!-- lower and upper is designated by radian-->
-	<limit effort="300" velocity="0.1" lower="-3.14" upper="3.14"/>
-	<dynamics daming="50" friction="1"/>
+    <parent link="base_link"/>
+    <child link="pan_link"/>
+    <origin xyz="0 0 0.1"/>
+    <axis xyz="0 0 1" />
+    <limit effort="300" velocity="0.1" lower="-3.14" upper="3.14"/>
+    <dynamics damping="50" friction="1"/>
   </joint>
   <link name="pan_link">
-	<visual>
-	  <geometry>
-		<cylinder length="${pan_link_length}" radius="${pan_link_radius}"/>
-	  </geometry>
-	  <origin rpy="0 0 0" xyz="0 0 0.9"/>
-	  <material name="red">
-		<color rgba="1 0 0 1"/>
-	  </material>
-	</visual>
-	<collision>
-		<geometry>
-		  <cylinder length="${pan_link_length}" radius="${pan_link_length+0.02}"/>
-		</geometry>
-		<origin rpy="0 0 0" xyz="0 0 0.09"/>
-	</collision>
+    <visual>
+      <geometry>
+	<cylinder length="${pan_link_length}" radius="${pan_link_radius}"/>
+      </geometry>
+      <origin rpy="0 0 0" xyz="0 0 0.09"/>
+      <material name="red">
+        <color rgba="0 0 1 1"/>
+      </material>
+    </visual>
+    <collision>
+      <geometry>
+	<cylinder length="${pan_link_length}" radius="${pan_link_radius+0.02}"/>
+      </geometry>
+      <origin rpy="0 0 0" xyz="0 0 0.09"/>
+    </collision>
 	<xacro:inertial_matrix mass="1"/>
   </link>
   <joint name="tilt_joint" type="revolute">
-	<parent link="pan_link"/>
-	<child link="tilt_link"/>
-	<origin xyz="0 0 0.2"/>
-	<axis xyz="0 1 0"/>
-	<limit effort="300" velocity="0.1" lower="-4.64" upper="-1.5"/>
-	<dynamics damping="50" friction="1"/>
+    <parent link="pan_link"/>
+    <child link="tilt_link"/>
+    <origin xyz="0 0 0.2"/>
+    <axis xyz="0 1 0" />
+    <limit effort="300" velocity="0.1" lower="-4.64" upper="-1.5"/>
+    <dynamics damping="50" friction="1"/>
   </joint>
   <link name="tilt_link">
-	<visual>
-	  <geometry>
-		<cylinder length="${tilt_link_length}" radius="${tilt_link_radius}"/>
-	  </geometry>
-	  <origin rpy="0 1.5 0" xyz="0 0 0"/>
-	  <material name="green">
-		<color rgba="1 0 0 1"/>
-	  </material>
-	</visual>
-	<collision>
-	  <geometry>
-		<cylinder length="${tilt_link_length}" radius="${tilt_link_radius+0.2}"/>
-	  </geometry>
-	  <origin rpy="0 1.5 0" xyz="0 0 0"/>
-	</collision>
+    <visual>
+      <geometry>
+	<cylinder length="${tilt_link_length}" radius="${tilt_link_radius}"/>
+      </geometry>
+      <origin rpy="0 1.5 0" xyz="0 0 0"/>
+      <material name="green">
+        <color rgba="1 0 0 1"/>
+      </material>
+    </visual>
+    <collision>
+      <geometry>
+	<cylinder length="${tilt_link_length}" radius="${tilt_link_radius+0.2}"/>
+      </geometry>
+      <origin rpy="0 1.5 0" xyz="0 0 0"/>
+    </collision>
 	<xacro:inertial_matrix mass="1"/>
   </link>

File: chapter2_codes/mastering_ros_robot_description_pkg/urdf/sensors/seven_dof_arm.xacro (robot description, xacro)
@@ -10,34 +10,34 @@
 	<color rgba="1 1 1 1"/>
   </material>
-  <property name="deg_to_rad" value="0.01745329251994329577"/>
+  <xacro:property name="deg_to_rad" value="0.01745329251994329577"/>
   <!-- Constants -->
-  <property name="M_SCALE" value="0.001 0.001 0.001 0.001"/>
-  <property name="M_PI" value="3.14159265398979"/>
-  <property name="shoulder_pan_width" value="0.04"/>
-  <property name="shoulder_pan_len" value="0.08"/>
-  <property name="shoulder_pitch_len" value="0.14"/>
-  <property name="shoulder_pitch_width" value="0.04"/>
-  <property name="shoulder_pitch_height" value="0.04"/>
-  <property name="elbow_roll_width" value="0.02"/>
-  <property name="elbow_roll_len" value="0.04"/>
-  <property name="elbow_pitch_len" value="0.22"/>
-  <property name="elbow_pitch_width" value="0.04"/>
-  <property name="elbow_pitch_height" value="0.04"/>
-  <property name="wrist_roll_width" value="0.02"/>
-  <property name="wrist_roll_len" value="0.04"/>
-  <property name="wrist_pitch_len" value="0.06"/>
-  <property name="wrist_pitch_width" value="0.04"/>
-  <property name="wrist_pitch_height" value="0.04"/>
-  <property name="gripper_roll_width" value="0.04"/>
-  <property name="gripper_roll_len" value="0.02"/>
-  <property name="left_gripper_len" value="0.08"/>
-  <property name="left_gripper_width" value="0.01"/>
-  <property name="left_gripper_height" value="0.01"/>
-  <property name="right_gripper_len" value="0.08"/>
-  <property name="right_gripper_width" value="0.01"/>
-  <property name="right_gripper_height" value="0.01"/>
-  <property name="grasp_frame_len" value="0.02"/>
-  <property name="grasp_frame_width" value="0.02"/>
-  <property name="grasp_frame_height" value="0.02"/>
+  <xacro:property name="M_SCALE" value="0.001 0.001 0.001 0.001"/>
+  <xacro:property name="M_PI" value="3.14159265398979"/>
+  <xacro:property name="shoulder_pan_width" value="0.04"/>
+  <xacro:property name="shoulder_pan_len" value="0.08"/>
+  <xacro:property name="shoulder_pitch_len" value="0.14"/>
+  <xacro:property name="shoulder_pitch_width" value="0.04"/>
+  <xacro:property name="shoulder_pitch_height" value="0.04"/>
+  <xacro:property name="elbow_roll_width" value="0.02"/>
+  <xacro:property name="elbow_roll_len" value="0.04"/>
+  <xacro:property name="elbow_pitch_len" value="0.22"/>
+  <xacro:property name="elbow_pitch_width" value="0.04"/>
+  <xacro:property name="elbow_pitch_height" value="0.04"/>
+  <xacro:property name="wrist_roll_width" value="0.02"/>
+  <xacro:property name="wrist_roll_len" value="0.04"/>
+  <xacro:property name="wrist_pitch_len" value="0.06"/>
+  <xacro:property name="wrist_pitch_width" value="0.04"/>
+  <xacro:property name="wrist_pitch_height" value="0.04"/>
+  <xacro:property name="gripper_roll_width" value="0.04"/>
+  <xacro:property name="gripper_roll_len" value="0.02"/>
+  <xacro:property name="left_gripper_len" value="0.08"/>
+  <xacro:property name="left_gripper_width" value="0.01"/>
+  <xacro:property name="left_gripper_height" value="0.01"/>
+  <xacro:property name="right_gripper_len" value="0.08"/>
+  <xacro:property name="right_gripper_width" value="0.01"/>
+  <xacro:property name="right_gripper_height" value="0.01"/>
+  <xacro:property name="grasp_frame_len" value="0.02"/>
+  <xacro:property name="grasp_frame_width" value="0.02"/>
+  <xacro:property name="grasp_frame_height" value="0.02"/>
   <xacro:macro name="inertial_matrix" params="mass">
 	<inertial>

File: chapter2_codes/mastering_ros_robot_description_pkg/urdf/sensors/xtion_pro_live.urdf.xacro (robot description, xacro)
@@ -14,5 +14,5 @@
     <!-- frames in the center of the camera -->
     <joint name="${name}_joint" type="fixed">
-      <insert_block name="origin"/>
+      <xacro:insert_block name="origin"/>
       <parent link="${parent}_link"/>
       <child link="${name}_link"/>
@@ -35,5 +35,5 @@
     </link>
     <joint name="${name}_optical_joint" type="fixed">
-      <insert_block name="optical_origin"/>
+      <xacro:insert_block name="optical_origin"/>
       <parent link="${name}_link"/>
       <child link="${name}_optical_frame"/>

File: chapter2_codes/mastering_ros_robot_description_pkg/urdf/seven_dof_arm.urdf (robot description, URDF)
Before this commit: robot seven_dof_arm, 12 links, 11 joints
Links:
- added link rgbd_camera_depth_frame, mass 0.001
- added link rgbd_camera_depth_optical_frame, mass 0.001
- added link rgbd_camera_link, mass 0.21970000000; visual mesh filename=package://mastering_ros_robot_description_pkg/meshes/sensor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
- added link rgbd_camera_optical_frame, mass 0.001
- added link rgbd_camera_rgb_frame, mass 0.001
- added link rgbd_camera_rgb_optical_frame, mass 0.001
- link elbow_roll_link: geometry collision cylinder length=0.06 radius=0.02; visual cylinder length=0.06 radius=0.02
- link grasping_frame: mass None -> 0.0001
- link wrist_roll_link: geometry collision cylinder length=0.06 radius=0.02; visual cylinder length=0.06 radius=0.02
Joints:
- removed joint finger_jiont2
- added joint finger_joint2: type prismatic, parent gripper_roll_link, child gripper_finger_link2, origin xyz=0.0 0 0, axis 0 1 0, limit lower=-0.03 upper=0 effort=1 velocity=1.0
- added joint rgbd_camera_depth_joint: type fixed, parent rgbd_camera_link, child rgbd_camera_depth_frame, origin xyz=0.0 0.049 0.0 rpy=0 0 0
- added joint rgbd_camera_depth_optical_joint: type fixed, parent rgbd_camera_depth_frame, child rgbd_camera_depth_optical_frame, origin xyz=0 0 0 rpy=-1.57079632679 0.0 -1.57079632679
- added joint rgbd_camera_joint: type fixed, parent base_link, child rgbd_camera_link, origin xyz=0.1 0 1 rpy=0 1.308996939 0
- added joint rgbd_camera_optical_joint: type fixed, parent rgbd_camera_link, child rgbd_camera_optical_frame, origin xyz=0 0 0 rpy=-1.57079632679 0 -1.57079632679
- added joint rgbd_camera_rgb_joint: type fixed, parent rgbd_camera_link, child rgbd_camera_rgb_frame, origin xyz=0.0 0.022 0.0 rpy=0 0 0
- added joint rgbd_camera_rgb_optical_joint: type fixed, parent rgbd_camera_rgb_frame, child rgbd_camera_rgb_optical_frame, origin xyz=0 0 0 rpy=-1.57079632679 0.0 -1.57079632679
- joint elbow_pitch_joint: limit lower=-1.59534 upper=1.9328 effort=300 velocity=1 -> lower=-1.5953400194 upper=1.93281579274 effort=300 velocity=1; origin xyz=-0.035 0 0.0 rpy=3.14159265399 1.57079632699 0 -> xyz=-0.035 0 0.0 rpy=0.055 1.570795 0
- joint elbow_roll_joint: limit lower=-2.61799 upper=0.70563 effort=300 velocity=1 -> lower=-2.61799387799 upper=0.705631162427 effort=300 velocity=1; origin xyz=-0.002 0 0.1206 rpy=3.14159265399 1.57079632699 0 -> xyz=-0.002 0 0.1206 rpy=3.14159 1.570795 0
- joint finger_joint1: limit lower=0 upper=0.03 effort=300 velocity=1.0 -> lower=0 upper=0.03 effort=100 velocity=1.0; origin xyz=0 0 0 -> xyz=0.0 0 0
- joint gripper_roll_joint: limit lower=-2.617993 upper=2.61288 effort=300 velocity=1 -> lower=-2.61799387799 upper=2.6128806087 effort=300 velocity=1; origin xyz=0 0 0.08 rpy=4.71238898098 -1.57079632699 0 -> xyz=0 0 0.080 rpy=4.712385 -1.570795 0
- joint shoulder_pan_joint: limit lower=-2.61799 upper=1.98394 effort=300 velocity=20 -> lower=-2.61799387799 upper=1.98394848567 effort=300 velocity=1; origin xyz=0 0 0.05 rpy=0 1.57079632699 0.0 -> xyz=0 0 0.05 rpy=0 1.570795 0.0
- joint shoulder_pitch_joint: limit lower=-1.1996 upper=1.8994 effort=300 velocity=1 -> lower=-1.19962513147 upper=1.89994105047 effort=300 velocity=1; origin xyz=-0.041 0.0021 0.0 rpy=-1.57079632699 0 1.57079632699 -> xyz=-0.041 0.0021 0.0 rpy=-1.570795 0 1.570795
- joint wrist_pitch_joint: limit lower=-1.59534 upper=1.98394 effort=300 velocity=1 -> lower=-1.5953400194 upper=1.98394848567 effort=300 velocity=1; origin xyz=0 0 0.0001 rpy=0 1.57079632699 0 -> xyz=0.0 0.0 0.0001 rpy=0 1.570795 0
- joint wrist_roll_joint: limit lower=-2.61799 upper=2.61288 effort=300 velocity=1 -> lower=-2.61799387799 upper=2.6128806087 effort=300 velocity=1; origin xyz=0.0 0.0081 -0.248 rpy=0 1.57079632699 3.14159265399 -> xyz=0.0 0.0081 -.248 rpy=0 1.570795 3.14159

File: chapter2_codes/mastering_ros_robot_description_pkg/urdf/seven_dof_arm.xacro (robot description, xacro)
@@ -1,4 +1,4 @@
 <?xml version="1.0"?>
-<robot name="seven_dof_arm" xmlns:xacro="http://www.ros.org/wiki/xacro">
+<robot name="seven_dof_arm" xmlns:xacro="http://ros.org/wiki/xacro">
   <!-- Include materials -->
     <material name="Black">
@@ -11,44 +11,44 @@
         <color rgba="1.0 1.0 1.0 1.0"/>
     </material>
-  <property name="deg_to_rad" value="0.01745329251994329577"/>
+  <xacro:property name="deg_to_rad" value="0.01745329251994329577"/>
   <!-- Constants -->
-  <property name="M_SCALE" value="0.001 0.001 0.001"/>
-  <property name="M_PI" value="3.14159"/>
+  <xacro:property name="M_SCALE" value="0.001 0.001 0.001"/>
+  <xacro:property name="M_PI" value="3.14159"/>
   <!-- Shoulder pan link properties -->
-  <property name="shoulder_pan_width" value="0.04" />
-  <property name="shoulder_pan_len" value="0.08" />
+  <xacro:property name="shoulder_pan_width" value="0.04" />
+  <xacro:property name="shoulder_pan_len" value="0.08" />
   <!-- Shoulder pitch link properties -->
-  <property name="shoulder_pitch_len" value="0.14" />
-  <property name="shoulder_pitch_width" value="0.04" />
-  <property name="shoulder_pitch_height" value="0.04" />
+  <xacro:property name="shoulder_pitch_len" value="0.14" />
+  <xacro:property name="shoulder_pitch_width" value="0.04" />
+  <xacro:property name="shoulder_pitch_height" value="0.04" />
   <!-- Elbow roll link properties -->
-  <property name="elbow_roll_width" value="0.02" />
-  <property name="elbow_roll_len" value="0.06" />
+  <xacro:property name="elbow_roll_width" value="0.02" />
+  <xacro:property name="elbow_roll_len" value="0.06" />
   <!-- Elbow pitch link properties -->
-  <property name="elbow_pitch_len" value="0.22" />
-  <property name="elbow_pitch_width" value="0.04" />
-  <property name="elbow_pitch_height" value="0.04" />
+  <xacro:property name="elbow_pitch_len" value="0.22" />
+  <xacro:property name="elbow_pitch_width" value="0.04" />
+  <xacro:property name="elbow_pitch_height" value="0.04" />
   <!-- Wrist roll link properties -->
-  <property name="wrist_roll_width" value="0.02" />
-  <property name="wrist_roll_len" value="0.04" />
+  <xacro:property name="wrist_roll_width" value="0.02" />
+  <xacro:property name="wrist_roll_len" value="0.04" />
   <!-- wrist pitch link properties -->
-  <property name="wrist_pitch_len" value="0.06" />
-  <property name="wrist_pitch_width" value="0.04" />
-  <property name="wrist_pitch_height" value="0.04" />
+  <xacro:property name="wrist_pitch_len" value="0.06" />
+  <xacro:property name="wrist_pitch_width" value="0.04" />
+  <xacro:property name="wrist_pitch_height" value="0.04" />
   <!-- Gripper roll link properties -->
-  <property name="gripper_roll_width" value="0.04" />
-  <property name="gripper_roll_len" value="0.02" />
+  <xacro:property name="gripper_roll_width" value="0.04" />
+  <xacro:property name="gripper_roll_len" value="0.02" />
   <!-- Left gripper -->
-  <property name="left_gripper_len" value="0.08" />
-  <property name="left_gripper_width" value="0.01" />
-  <property name="left_gripper_height" value="0.01" />
+  <xacro:property name="left_gripper_len" value="0.08" />
+  <xacro:property name="left_gripper_width" value="0.01" />
+  <xacro:property name="left_gripper_height" value="0.01" />
   <!-- Right gripper -->
-  <property name="right_gripper_len" value="0.08" />
-  <property name="right_gripper_width" value="0.01" />
-  <property name="right_gripper_height" value="0.01" />
+  <xacro:property name="right_gripper_len" value="0.08" />
+  <xacro:property name="right_gripper_width" value="0.01" />
+  <xacro:property name="right_gripper_height" value="0.01" />
   <!-- Right gripper -->
-  <property name="grasp_frame_len" value="0.02" />
-  <property name="grasp_frame_width" value="0.02" />
-  <property name="grasp_frame_height" value="0.02" />
+  <xacro:property name="grasp_frame_len" value="0.02" />
+  <xacro:property name="grasp_frame_width" value="0.02" />
+  <xacro:property name="grasp_frame_height" value="0.02" />
    <xacro:macro name="inertial_matrix" params="mass">
       <inertial>

File: chapter2_codes/mastering_ros_robot_description_pkg/urdf/wheel.urdf.xacro (robot description, xacro)
@@ -2,15 +2,15 @@
 <robot name="wheel" xmlns:xacro="http://www.ros.org/wiki/xacro">
   <!-- Wheels -->
-  <property name="wheel_radius" value="0.04" />
-  <property name="wheel_height" value="0.02" />
-  <property name="wheel_mass" value="2.5" /> <!-- in kg-->
-  <property name="base_x_origin_to_wheel_origin" value="0.25" />
-  <property name="base_y_origin_to_wheel_origin" value="0.3" />
-  <property name="base_z_origin_to_wheel_origin" value="0.0" />
-  <macro name="cylinder_inertia" params="m r h">
+  <xacro:property name="wheel_radius" value="0.04" />
+  <xacro:property name="wheel_height" value="0.02" />
+  <xacro:property name="wheel_mass" value="2.5" /> <!-- in kg-->
+  <xacro:property name="base_x_origin_to_wheel_origin" value="0.25" />
+  <xacro:property name="base_y_origin_to_wheel_origin" value="0.3" />
+  <xacro:property name="base_z_origin_to_wheel_origin" value="0.0" />
+  <xacro:macro name="cylinder_inertia" params="m r h">
     <inertia  ixx="${m*(3*r*r+h*h)/12}" ixy = "0" ixz = "0"
               iyy="${m*(3*r*r+h*h)/12}" iyz = "0"
               izz="${m*r*r/2}" />
-  </macro>
+  </xacro:macro>
   <xacro:macro name="wheel" params="fb lr parent translateX translateY flipY"> <!--fb : front, back ; lr: left, right -->
     <link name="${fb}_${lr}_wheel">
