Commit message: checked chapter3/ch3_seven_dof_arm_gazebo

File: chapter3_codes/ch3_seven_dof_arm_gazebo/urdf/ch3_seven_dof_arm_gazebo.xacro (robot description, xacro)
@@ -1,4 +1,4 @@
 <?xml version="1.0"?>
-<robot name="ch3_seven_dof_arm_gazebo" xmlns:xacro="http://www.ros.org/wiki/xacro">
+<robot name="seven_dof_arm" xmlns:xacro="http://ros.org/wiki/xacro">
   <!-- Include materials -->
     <material name="Black">
@@ -11,44 +11,44 @@
         <color rgba="1.0 1.0 1.0 1.0"/>
     </material>
-  <property name="deg_to_rad" value="0.01745329251994329577"/>
+  <xacro:property name="deg_to_rad" value="0.01745329251994329577"/>
   <!-- Constants -->
-  <property name="M_SCALE" value="0.001 0.001 0.001"/>
-  <property name="M_PI" value="3.14159"/>
+  <xacro:property name="M_SCALE" value="0.001 0.001 0.001"/>
+  <xacro:property name="M_PI" value="3.14159"/>
   <!-- Shoulder pan link properties -->
-  <property name="shoulder_pan_width" value="0.04" />
-  <property name="shoulder_pan_len" value="0.08" />
+  <xacro:property name="shoulder_pan_width" value="0.04" />
+  <xacro:property name="shoulder_pan_len" value="0.08" />
   <!-- Shoulder pitch link properties -->
-  <property name="shoulder_pitch_len" value="0.14" />
-  <property name="shoulder_pitch_width" value="0.04" />
-  <property name="shoulder_pitch_height" value="0.04" />
+  <xacro:property name="shoulder_pitch_len" value="0.14" />
+  <xacro:property name="shoulder_pitch_width" value="0.04" />
+  <xacro:property name="shoulder_pitch_height" value="0.04" />
   <!-- Elbow roll link properties -->
-  <property name="elbow_roll_width" value="0.02" />
-  <property name="elbow_roll_len" value="0.06" />
+  <xacro:property name="elbow_roll_width" value="0.02" />
+  <xacro:property name="elbow_roll_len" value="0.06" />
   <!-- Elbow pitch link properties -->
-  <property name="elbow_pitch_len" value="0.22" />
-  <property name="elbow_pitch_width" value="0.04" />
-  <property name="elbow_pitch_height" value="0.04" />
+  <xacro:property name="elbow_pitch_len" value="0.22" />
+  <xacro:property name="elbow_pitch_width" value="0.04" />
+  <xacro:property name="elbow_pitch_height" value="0.04" />
   <!-- Wrist roll link properties -->
-  <property name="wrist_roll_width" value="0.02" />
-  <property name="wrist_roll_len" value="0.04" />
+  <xacro:property name="wrist_roll_width" value="0.02" />
+  <xacro:property name="wrist_roll_len" value="0.04" />
   <!-- wrist pitch link properties -->
-  <property name="wrist_pitch_len" value="0.06" />
-  <property name="wrist_pitch_width" value="0.04" />
-  <property name="wrist_pitch_height" value="0.04" />
+  <xacro:property name="wrist_pitch_len" value="0.06" />
+  <xacro:property name="wrist_pitch_width" value="0.04" />
+  <xacro:property name="wrist_pitch_height" value="0.04" />
   <!-- Gripper roll link properties -->
-  <property name="gripper_roll_width" value="0.04" />
-  <property name="gripper_roll_len" value="0.02" />
+  <xacro:property name="gripper_roll_width" value="0.04" />
+  <xacro:property name="gripper_roll_len" value="0.02" />
   <!-- Left gripper -->
-  <property name="left_gripper_len" value="0.08" />
-  <property name="left_gripper_width" value="0.01" />
-  <property name="left_gripper_height" value="0.01" />
+  <xacro:property name="left_gripper_len" value="0.08" />
+  <xacro:property name="left_gripper_width" value="0.01" />
+  <xacro:property name="left_gripper_height" value="0.01" />
   <!-- Right gripper -->
-  <property name="right_gripper_len" value="0.08" />
-  <property name="right_gripper_width" value="0.01" />
-  <property name="right_gripper_height" value="0.01" />
+  <xacro:property name="right_gripper_len" value="0.08" />
+  <xacro:property name="right_gripper_width" value="0.01" />
+  <xacro:property name="right_gripper_height" value="0.01" />
   <!-- Right gripper -->
-  <property name="grasp_frame_len" value="0.02" />
-  <property name="grasp_frame_width" value="0.02" />
-  <property name="grasp_frame_height" value="0.02" />
+  <xacro:property name="grasp_frame_len" value="0.02" />
+  <xacro:property name="grasp_frame_width" value="0.02" />
+  <xacro:property name="grasp_frame_height" value="0.02" />
    <xacro:macro name="inertial_matrix" params="mass">
       <inertial>
@@ -58,6 +58,5 @@
    </xacro:macro>
    <!--
-	   Deprecated syntax, please prepend 'hardware_interface/' to'PositionJointInterface' within the <hardwareInterface> tag in joint 'shoulder_pan_joint'.
-	   というエラーが出た
+	   Deprecated syntax, please prepend 'hardware_interface/' to'PositionJointInterface' within the <hardwareInterface> tag in joint 'shoulder_pan_joint'
    -->
    <xacro:macro name="transmission_block" params="joint_name">
@@ -420,4 +419,5 @@
     <plugin name="gazebo_ros_control" filename="libgazebo_ros_control.so">
       <robotNamespace>/ch3_seven_dof_arm_gazebo</robotNamespace>
+	  <legacyModeNS>true</legacyModeNS>
     </plugin>
   </gazebo>

File: chapter3_codes/ch3_seven_dof_arm_gazebo/urdf/sensors/xtion_pro_live.urdf.xacro (robot description, xacro)
@@ -1,5 +1,5 @@
 <?xml version="1.0"?>
 <robot xmlns:xacro="http://ros.org/wiki/xacro">
-  <xacro:include filename="$(find mastering_ros_robot_description_pkg)/urdf/sensors/xtion_pro_live.gazebo.xacro"/>
+  <xacro:include filename="$(find ch3_seven_dof_arm_gazebo)/urdf/sensors/xtion_pro_live.gazebo.xacro"/>
   <xacro:macro name="dummy_inertial">
     <inertial>
@@ -14,5 +14,5 @@
     <!-- frames in the center of the camera -->
     <joint name="${name}_joint" type="fixed">
-      <insert_block name="origin"/>
+      <xacro:insert_block name="origin"/>
       <parent link="${parent}_link"/>
       <child link="${name}_link"/>
@@ -29,5 +29,5 @@
         <origin xyz="0 0 0" rpy="0 0 0"/>
         <geometry>
-          <mesh filename="package://mastering_ros_robot_description_pkg/meshes/sensors/xtion_pro_live/xtion_pro_live.dae"/>
+          <mesh filename="package://ch3_seven_dof_arm_gazebo/meshes/sensors/xtion_pro_live/xtion_pro_live.dae"/>
         </geometry>
         <material name="DarkGrey"/>
@@ -35,5 +35,5 @@
     </link>
     <joint name="${name}_optical_joint" type="fixed">
-      <insert_block name="optical_origin"/>
+      <xacro:insert_block name="optical_origin"/>
       <parent link="${name}_link"/>
       <child link="${name}_optical_frame"/>
