Commit message: started ch4_diff_wheeled_robot

File: chapter4_codes/ch4_seven_dof_arm_config/urdf/ch4_seven_dof_arm_gazebo.xacro (robot description, xacro)
@@ -2,13 +2,13 @@
 <robot name="seven_dof_arm" xmlns:xacro="http://ros.org/wiki/xacro">
   <!-- Include materials -->
-    <material name="Black">
-        <color rgba="0.0 0.0 0.0 1.0"/>
-    </material>
-    <material name="Red">
-        <color rgba="0.8 0.0 0.0 1.0"/>
-    </material>
-    <material name="White">
-        <color rgba="1.0 1.0 1.0 1.0"/>
-    </material>
+  <material name="Black">
+    <color rgba="0.0 0.0 0.0 1.0"/>
+  </material>
+  <material name="Red">
+    <color rgba="0.8 0.0 0.0 1.0"/>
+  </material>
+  <material name="White">
+    <color rgba="1.0 1.0 1.0 1.0"/>
+  </material>
   <xacro:property name="deg_to_rad" value="0.01745329251994329577"/>
   <!-- Constants -->
@@ -51,28 +51,33 @@
   <xacro:property name="grasp_frame_width" value="0.02" />
   <xacro:property name="grasp_frame_height" value="0.02" />
-   <xacro:macro name="inertial_matrix" params="mass">
-      <inertial>
-      	<mass value="${mass}" />
-        <inertia ixx="1.0" ixy="0.0" ixz="0.0" iyy="0.5" iyz="0.0" izz="1.0" />
-      </inertial>
-   </xacro:macro>
-   <!--
-	   Deprecated syntax, please prepend 'hardware_interface/' to'PositionJointInterface' within the <hardwareInterface> tag in joint 'shoulder_pan_joint'
-   -->
-   <xacro:macro name="transmission_block" params="joint_name">
-	  <transmission name="tran1">
-	    <type>transmission_interface/SimpleTransmission</type>
-	    <joint name="${joint_name}">
-	      <hardwareInterface>hardware_interface/PositionJointInterface</hardwareInterface>
-	    </joint>
-	    <actuator name="motor1">
-	      <mechanicalReduction>1</mechanicalReduction>
-	    </actuator>
-	  </transmission>
-   </xacro:macro>
-<!-- BOTTOM FIXED LINK
-This link is the base of the arm in which arm is placed
--->
-<!-- ///////////////////////////////////////////////////////////////////////////////////////////////////////////////////// -->
+  <xacro:macro name="inertial_matrix" params="mass">
+    <inertial>
+      <mass value="${mass}" />
+      <inertia ixx="1.0" ixy="0.0" ixz="0.0" iyy="0.5" iyz="0.0" izz="1.0" />
+    </inertial>
+  </xacro:macro>
+  <!--
+	  Deprecated syntax, please prepend 'hardware_interface/' to'PositionJointInterface' within the <hardwareInterface> tag in joint 'shoulder_pan_joint'
+  -->
+  <xacro:macro name="transmission_block" params="joint_name">
+	<transmission name="tran1">
+	  <type>transmission_interface/SimpleTransmission</type>
+	  <joint name="${joint_name}">
+	    <hardwareInterface>hardware_interface/PositionJointInterface</hardwareInterface>
+	  </joint>
+	  <actuator name="motor1">
+	    <mechanicalReduction>1</mechanicalReduction>
+	  </actuator>
+	</transmission>
+  </xacro:macro>
+  <!-- BOTTOM FIXED LINK
+	   This link is the base of the arm in which arm is placed
+  -->
+  <!-- ///////////////////////////////////////////////////////////////////////////////////////////////////////////////////// -->
+  <link name="world"/>
+  <joint name="bottom_world_joint" type="fixed">
+	<parent link="world"/>
+	<child link="base_link"/>
+  </joint>
   <joint name="bottom_joint" type="fixed">
     <origin xyz="0 0 0" rpy="0 0 0" />
@@ -84,5 +89,5 @@
       <origin xyz=" 0 0 -0.04"  rpy="0 0 0"/>
       <geometry>
-	       <box size="1 1 0.02" />
+	    <box size="1 1 0.02" />
       </geometry>
       <material name="Brown" />
@@ -91,5 +96,5 @@
       <origin xyz=" 0 0 -0.04"  rpy="0 0 0"/>
       <geometry>
-	       <box size="1 1 0.02" />
+	    <box size="1 1 0.02" />
       </geometry>
       </collision>>
@@ -98,5 +103,5 @@
     <material>Gazebo/White</material>
   </gazebo>
-<!-- ///////////////////////////////////////////////////////////////////////////////////////////////////////////////////// -->
+  <!-- ///////////////////////////////////////////////////////////////////////////////////////////////////////////////////// -->
   <!-- BASE LINK -->
   <link name="base_link">
@@ -104,5 +109,5 @@
       <origin xyz="0 0 0" rpy="${M_PI/2} 0 0" /> <!-- rotate PI/2 -->
       <geometry>
-	       <box size="0.1 0.1 0.1" />
+	    <box size="0.1 0.1 0.1" />
       </geometry>
       <material name="White" />
@@ -111,8 +116,8 @@
       <origin xyz="0 0 0" rpy="${M_PI/2} 0 0" /> <!-- rotate PI/2 -->
       <geometry>
-	       <box size="0.1 0.1 0.1" />
+	    <box size="0.1 0.1 0.1" />
       </geometry>
       </collision>>
-	<xacro:inertial_matrix mass="1"/>
+	  <xacro:inertial_matrix mass="1"/>
   </link>
   <gazebo reference="base_link">
@@ -127,5 +132,5 @@
     <dynamics damping="50" friction="1"/>
   </joint>
-<!-- ///////////////////////////////////////////////////////////////////////////////////////////////////////////////////// -->
+  <!-- ///////////////////////////////////////////////////////////////////////////////////////////////////////////////////// -->
   <!-- SHOULDER PAN LINK -->
   <link name="shoulder_pan_link" >
@@ -133,5 +138,5 @@
       <origin xyz="0 0 0" rpy="0 ${M_PI/2} 0" />
       <geometry>
-            <cylinder radius="${shoulder_pan_width}" length="${shoulder_pan_len}"/>
+        <cylinder radius="${shoulder_pan_width}" length="${shoulder_pan_len}"/>
       </geometry>
       <material name="Red" />
@@ -140,5 +145,5 @@
       <origin xyz="0 0 0" rpy="0 ${M_PI/2} 0" />
       <geometry>
-            <cylinder radius="${shoulder_pan_width}" length="${shoulder_pan_len}"/>
+        <cylinder radius="${shoulder_pan_width}" length="${shoulder_pan_len}"/>
       </geometry>
     </collision>
@@ -156,12 +161,12 @@
     <dynamics damping="50" friction="1"/>
   </joint>
-<!-- ///////////////////////////////////////////////////////////////////////////////////////////////////////////////////// -->
-<!-- SHOULDER PITCH LINK -->
-<!-- rotate on z axis -->
+  <!-- ///////////////////////////////////////////////////////////////////////////////////////////////////////////////////// -->
+  <!-- SHOULDER PITCH LINK -->
+  <!-- rotate on z axis -->
   <link name="shoulder_pitch_link" >
     <visual>
       <origin xyz="-0.002 0 0.04" rpy="0 ${M_PI/2} 0" />
       <geometry>
-           <box size="${shoulder_pitch_len} ${shoulder_pitch_width} ${shoulder_pitch_height}" />
+        <box size="${shoulder_pitch_len} ${shoulder_pitch_width} ${shoulder_pitch_height}" />
       </geometry>
       <material name="White" />
@@ -170,5 +175,5 @@
       <origin xyz="-0.002 0 0.04" rpy="0 ${M_PI/2} 0" />
       <geometry>
-           <box size="${shoulder_pitch_len} ${shoulder_pitch_width} ${shoulder_pitch_height}" />
+        <box size="${shoulder_pitch_len} ${shoulder_pitch_width} ${shoulder_pitch_height}" />
       </geometry>
     </collision>
@@ -186,5 +191,5 @@
     <dynamics damping="50" friction="1"/>
   </joint>
-<!-- ///////////////////////////////////////////////////////////////////////////////////////////////////////////////////// -->
+  <!-- ///////////////////////////////////////////////////////////////////////////////////////////////////////////////////// -->
   <!-- ELBOW ROLL LINK -->
   <link name="elbow_roll_link" >
@@ -192,5 +197,5 @@
       <origin xyz="-0.015 0.0 -0.0" rpy="0 ${M_PI/2} 0" />
       <geometry>
-            <cylinder radius="${elbow_roll_width}" length="${elbow_roll_len}"/>
+        <cylinder radius="${elbow_roll_width}" length="${elbow_roll_len}"/>
       </geometry>
       <material name="Black" />
@@ -199,5 +204,5 @@
       <origin xyz="-0.015 0.0 -0.0" rpy="0 ${M_PI/2} 0" />
       <geometry>
-            <cylinder radius="${elbow_roll_width}" length="${elbow_roll_len}"/>
+        <cylinder radius="${elbow_roll_width}" length="${elbow_roll_len}"/>
       </geometry>
     </collision>
@@ -215,5 +220,5 @@
     <dynamics damping="50" friction="1"/>
   </joint>
-<!-- ///////////////////////////////////////////////////////////////////////////////////////////////////////////////////// -->
+  <!-- ///////////////////////////////////////////////////////////////////////////////////////////////////////////////////// -->
   <!-- ELBOW PITCH LINK -->
   <link name="elbow_pitch_link" >
@@ -221,5 +226,5 @@
       <origin xyz="0 0 -0.12" rpy="0 ${M_PI/2} 0" />
       <geometry>
-       <box size="${elbow_pitch_len} ${elbow_pitch_width} ${elbow_pitch_height}" />
+		<box size="${elbow_pitch_len} ${elbow_pitch_width} ${elbow_pitch_height}" />
       </geometry>
       <material name="Red" />
@@ -228,5 +233,5 @@
       <origin xyz="0 0 -0.12" rpy="0 ${M_PI/2} 0" />
       <geometry>
-       <box size="${elbow_pitch_len} ${elbow_pitch_width} ${elbow_pitch_height}" />
+		<box size="${elbow_pitch_len} ${elbow_pitch_width} ${elbow_pitch_height}" />
       </geometry>
     </collision>
@@ -249,5 +254,5 @@
       <origin xyz="0 0 0" rpy="0 ${M_PI/2} 0" />
       <geometry>
-           <cylinder radius="${elbow_roll_width}" length="${elbow_roll_len}"/>
+        <cylinder radius="${elbow_roll_width}" length="${elbow_roll_len}"/>
       </geometry>
       <material name="Black" />
@@ -256,5 +261,5 @@
       <origin xyz="0 0 0" rpy="0 ${M_PI/2} 0" />
       <geometry>
-           <cylinder radius="${elbow_roll_width}" length="${elbow_roll_len}"/>
+        <cylinder radius="${elbow_roll_width}" length="${elbow_roll_len}"/>
       </geometry>
     </collision>
@@ -272,5 +277,5 @@
     <dynamics damping="50" friction="1"/>
   </joint>
-<!-- ///////////////////////////////////////////////////////////////////////////////////////////////////////////////////// -->
+  <!-- ///////////////////////////////////////////////////////////////////////////////////////////////////////////////////// -->
   <!-- WRIST PITCH LINK -->
   <link name="wrist_pitch_link">
@@ -278,5 +283,5 @@
       <origin xyz="0 0 0.04" rpy="0 ${M_PI/2} 0" />
       <geometry>
-           <box size="${wrist_pitch_len} ${wrist_pitch_width} ${wrist_pitch_height}" />
+        <box size="${wrist_pitch_len} ${wrist_pitch_width} ${wrist_pitch_height}" />
       </geometry>
       <material name="White" />
@@ -285,5 +290,5 @@
       <origin xyz="0 0 0.04 " rpy="0 ${M_PI/2} 0" />
       <geometry>
-          <box size="${wrist_pitch_len} ${wrist_pitch_width} ${wrist_pitch_height}" />
+        <box size="${wrist_pitch_len} ${wrist_pitch_width} ${wrist_pitch_height}" />
       </geometry>
     </collision>
@@ -301,5 +306,5 @@
     <dynamics damping="50" friction="1"/>
   </joint>
-<!-- ///////////////////////////////////////////////////////////////////////////////////////////////////////////////////// -->
+  <!-- ///////////////////////////////////////////////////////////////////////////////////////////////////////////////////// -->
   <!-- GRIPPER ROLL LINK -->
   <link name="gripper_roll_link">
@@ -307,5 +312,5 @@
       <origin xyz="0 0 0" rpy="0 ${M_PI/2} 0" />
       <geometry>
-            <cylinder radius="${gripper_roll_width}" length="${gripper_roll_len}"/>
+        <cylinder radius="${gripper_roll_width}" length="${gripper_roll_len}"/>
       </geometry>
       <material name="Red" />
@@ -314,5 +319,5 @@
       <origin xyz="0 0 0" rpy="0 ${M_PI/2} 0" />
       <geometry>
-            <cylinder radius="${gripper_roll_width}" length="${gripper_roll_len}"/>
+        <cylinder radius="${gripper_roll_width}" length="${gripper_roll_len}"/>
       </geometry>
     </collision>
@@ -327,18 +332,18 @@
     <origin xyz="0.0 0 0" />
     <axis xyz="0 1 0" />
-      <limit effort="100" lower="0" upper="0.03" velocity="1.0"/>
-      <safety_controller k_position="20"
-                         k_velocity="20"
-                         soft_lower_limit="${-0.15 }"
-                         soft_upper_limit="${ 0.0 }"/>
-    <dynamics damping="50" friction="1"/>
-  </joint>
-<!-- ///////////////////////////////////////////////////////////////////////////////////////////////////////////////////// -->
+    <limit effort="100" lower="0" upper="0.03" velocity="1.0"/>
+    <safety_controller k_position="20"
+                       k_velocity="20"
+                       soft_lower_limit="${-0.15 }"
+                       soft_upper_limit="${ 0.0 }"/>
+    <dynamics damping="50" friction="1"/>
+  </joint>
+  <!-- ///////////////////////////////////////////////////////////////////////////////////////////////////////////////////// -->
   <!-- LEFT GRIPPER AFT LINK -->
   <link name="gripper_finger_link1">
-     <visual>
+    <visual>
       <origin xyz="0.04 -0.03 0"/>
       <geometry>
-           <box size="${left_gripper_len} ${left_gripper_width} ${left_gripper_height}" />
+        <box size="${left_gripper_len} ${left_gripper_width} ${left_gripper_height}" />
       </geometry>
       <material name="White" />
@@ -349,5 +354,5 @@
     <material>Gazebo/White</material>
   </gazebo>
-<!-- Joint between Wrist roll and finger 2 -->
+  <!-- Joint between Wrist roll and finger 2 -->
   <joint name="finger_joint2" type="prismatic">
     <parent link="gripper_roll_link"/>
@@ -356,8 +361,8 @@
     <axis xyz="0 1 0" />
     <limit effort="1" lower="-0.03" upper="0" velocity="1.0"/>
-<!--    <mimic joint="gripper_finger_joint" multiplier="-1.0" offset="0.0" /> -->
-    <dynamics damping="50" friction="1"/>
-  </joint>
-<!-- ///////////////////////////////////////////////////////////////////////////////////////////////////////////////////// -->
+	<!--    <mimic joint="gripper_finger_joint" multiplier="-1.0" offset="0.0" /> -->
+    <dynamics damping="50" friction="1"/>
+  </joint>
+  <!-- ///////////////////////////////////////////////////////////////////////////////////////////////////////////////////// -->
   <!-- RIGHT GRIPPER AFT LINK -->
   <link name="gripper_finger_link2">
@@ -365,5 +370,5 @@
       <origin xyz="0.04 0.03 0"/>
       <geometry>
-          <box size="${right_gripper_len} ${right_gripper_width} ${right_gripper_height}" />
+        <box size="${right_gripper_len} ${right_gripper_width} ${right_gripper_height}" />
       </geometry>
       <material name="White" />
@@ -374,46 +379,46 @@
     <material>Gazebo/White</material>
   </gazebo>
-    <!-- Grasping frame -->
-    <link name="grasping_frame">
-      <inertial>
-        <origin xyz="0 0 0" rpy="0 0 0"/>
-        <mass value="0.0001"/>
-        <cuboid_inertia mass="0.0001" x="0.001" y="0.001" z="0.001"/>
-        <inertia  ixx="1.0" ixy="0.0"  ixz="0.0"  iyy="100.0"  iyz="0.0"  izz="1.0" />
-      </inertial>
+  <!-- Grasping frame -->
+  <link name="grasping_frame">
+    <inertial>
+      <origin xyz="0 0 0" rpy="0 0 0"/>
+      <mass value="0.0001"/>
+      <cuboid_inertia mass="0.0001" x="0.001" y="0.001" z="0.001"/>
+      <inertia  ixx="1.0" ixy="0.0"  ixz="0.0"  iyy="100.0"  iyz="0.0"  izz="1.0" />
+    </inertial>
     <visual>
       <origin xyz="0 0 0"/>
       <geometry>
-          <box size="${grasp_frame_len} ${grasp_frame_width} ${grasp_frame_height}" />
-      </geometry>
-      <material name="White" />
-    </visual>
-    </link>
-    <joint name="grasping_frame_joint" type="fixed">
-      <parent link="gripper_roll_link"/>
-      <child link="grasping_frame"/>
-      <origin xyz="0.08 0 0" rpy="0 0 0"/>
-    </joint>
+        <box size="${grasp_frame_len} ${grasp_frame_width} ${grasp_frame_height}" />
+      </geometry>
+      <material name="White" />
+    </visual>
+  </link>
+  <joint name="grasping_frame_joint" type="fixed">
+    <parent link="gripper_roll_link"/>
+    <child link="grasping_frame"/>
+    <origin xyz="0.08 0 0" rpy="0 0 0"/>
+  </joint>
   <xacro:include filename="$(find ch4_seven_dof_arm_config)/urdf/sensors/xtion_pro_live.urdf.xacro"/>
-<!-- ///////////////////////////////////////////////////////////////////////////////////////////////////////////////////// -->
+  <!-- ///////////////////////////////////////////////////////////////////////////////////////////////////////////////////// -->
   <!-- Transmissions for ROS Control -->
-   <xacro:transmission_block joint_name="shoulder_pan_joint"/>
-   <xacro:transmission_block joint_name="shoulder_pitch_joint"/>
-   <xacro:transmission_block joint_name="elbow_roll_joint"/>
-   <xacro:transmission_block joint_name="elbow_pitch_joint"/>
-   <xacro:transmission_block joint_name="wrist_roll_joint"/>
-   <xacro:transmission_block joint_name="wrist_pitch_joint"/>
-   <xacro:transmission_block joint_name="gripper_roll_joint"/>
-   <xacro:transmission_block joint_name="finger_joint1"/>
-   <xacro:transmission_block joint_name="finger_joint2"/>
-<!--
-  <xacro:base name="base"/>
-  <xacro:arm parent="base"/>
-  <xacro:gripper parent="tool"/>
--->
-   <xacro:xtion_pro_live name="rgbd_camera" parent="base">
+  <xacro:transmission_block joint_name="shoulder_pan_joint"/>
+  <xacro:transmission_block joint_name="shoulder_pitch_joint"/>
+  <xacro:transmission_block joint_name="elbow_roll_joint"/>
+  <xacro:transmission_block joint_name="elbow_pitch_joint"/>
+  <xacro:transmission_block joint_name="wrist_roll_joint"/>
+  <xacro:transmission_block joint_name="wrist_pitch_joint"/>
+  <xacro:transmission_block joint_name="gripper_roll_joint"/>
+  <xacro:transmission_block joint_name="finger_joint1"/>
+  <xacro:transmission_block joint_name="finger_joint2"/>
+  <!--
+	  <xacro:base name="base"/>
+	  <xacro:arm parent="base"/>
+	  <xacro:gripper parent="tool"/>
+  -->
+  <xacro:xtion_pro_live name="rgbd_camera" parent="base">
     <origin xyz="0.1 0 1" rpy="0 ${75.0 * deg_to_rad} 0"/>
     <origin xyz="0 0 0" rpy="${-90.0 * deg_to_rad} 0 ${-90.0 * deg_to_rad}"/>
-   </xacro:xtion_pro_live>
+  </xacro:xtion_pro_live>
   <gazebo>
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