Commit message: chapter4: succeeded in loading worlds/ch4-willowgarage.world

File: chapter4_codes/ch4_diff_wheeled_robot/urdf/diff_wheeled_robot.xacro (robot description, xacro)
@@ -2,5 +2,5 @@
 <robot name="differential_wheeled_robot" xmlns:xacro="http://ros.org/wiki/xacro">
   <xacro:include filename="$(find ch4_diff_wheeled_robot)/urdf/wheel.urdf.xacro" />
-<!-- Defining the colors used in this robot -->
+  <!-- Defining the colors used in this robot -->
   <material name="Black">
     <color rgba="0.0 0.0 0.0 1.0"/>
@@ -55,12 +55,12 @@
       <origin xyz="0 0 0" />
       <inertia ixx="0.0001" ixy="0.0" ixz="0.0"
-          iyy="0.0001" iyz="0.0"
-          izz="0.0001" />
-    </inertial>
-    <visual>
-        <origin xyz="0 0 0" rpy="0 0 0" />
-        <geometry>
-            <box size="0.001 0.001 0.001" />
-        </geometry>
+			   iyy="0.0001" iyz="0.0"
+			   izz="0.0001" />
+    </inertial>
+    <visual>
+      <origin xyz="0 0 0" rpy="0 0 0" />
+      <geometry>
+        <box size="0.001 0.001 0.001" />
+      </geometry>
     </visual>
   </link>
@@ -80,10 +80,10 @@
       <origin xyz="0 0 0" />
       <!--The 3x3 rotational inertia matrix. -->
-        <cylinder_inertia  m="${base_mass}" r="${base_radius}" h="${base_height}" />
+      <cylinder_inertia  m="${base_mass}" r="${base_radius}" h="${base_height}" />
     </inertial>
     <visual>
       <origin xyz="0 0 0" rpy="0 0 0" />
       <geometry>
-          <cylinder length="${base_height}" radius="${base_radius}" />
+        <cylinder length="${base_height}" radius="${base_radius}" />
       </geometry>
       <material name="White" />
@@ -92,5 +92,5 @@
       <origin xyz="0 0 0" rpy="0 0 0 " />
       <geometry>
-          <cylinder length="${base_height}" radius="${base_radius}" />
+        <cylinder length="${base_height}" radius="${base_radius}" />
       </geometry>
     </collision>
@@ -100,67 +100,67 @@
     <turnGravityOff>false</turnGravityOff>
   </gazebo>
-<!--Caster front  -->
-    <link name="caster_front_link">
+  <!--Caster front  -->
+  <link name="caster_front_link">
     <visual>
       <origin xyz="0 0.02 0" rpy="${M_PI/2} 0 0" />
       <geometry>
-	<sphere radius="${caster_f_radius}" />
+		<sphere radius="${caster_f_radius}" />
       </geometry>
       <material name="Black" />
     </visual>
-      <collision>
-        <geometry>
-	<sphere radius="${caster_f_radius}" />
-        </geometry>
+    <collision>
+      <geometry>
+		<sphere radius="${caster_f_radius}" />
+      </geometry>
       <origin xyz="0 0.02 0" rpy="${M_PI/2} 0 0" />
-      </collision>
-      <inertial>
-        <mass value="${caster_f_mass}" />
-        <origin xyz="0 0 0" />
-        <inertia ixx="0.001" ixy="0.0" ixz="0.0"
-                 iyy="0.001" iyz="0.0"
-                 izz="0.001" />
-      </inertial>
-    </link>
- <joint name="caster_front_joint" type="fixed">
-      <parent link="base_link"/>
-      <child link="caster_front_link"/>
-      <origin xyz="0.115 0.0 0.007" rpy="${-M_PI/2} 0 0"/>
-    </joint>
+    </collision>
+    <inertial>
+      <mass value="${caster_f_mass}" />
+      <origin xyz="0 0 0" />
+      <inertia ixx="0.001" ixy="0.0" ixz="0.0"
+               iyy="0.001" iyz="0.0"
+               izz="0.001" />
+    </inertial>
+  </link>
+  <joint name="caster_front_joint" type="fixed">
+    <parent link="base_link"/>
+    <child link="caster_front_link"/>
+    <origin xyz="0.115 0.0 0.007" rpy="${-M_PI/2} 0 0"/>
+  </joint>
   <gazebo reference="caster_front_link">
     <turnGravityOff>false</turnGravityOff>
   </gazebo>
-<!--Caster back  -->
-    <link name="caster_back_link">
+  <!--Caster back  -->
+  <link name="caster_back_link">
     <visual>
       <origin xyz="0.02 0.02 0 " rpy="${M_PI/2} 0 0" />
       <geometry>
-	<sphere radius="${caster_b_radius}" />
+		<sphere radius="${caster_b_radius}" />
       </geometry>
       <material name="Black" />
     </visual>
-      <collision>
-        <geometry>
+    <collision>
+      <geometry>
 		<sphere radius="${caster_b_radius}" />
-        </geometry>
+      </geometry>
       <origin xyz="0 0.02 0 " rpy="${M_PI/2} 0 0" />
-      </collision>
-      <inertial>
-        <mass value="${caster_b_mass}" />
-        <origin xyz="0 0 0" />
-        <inertia ixx="0.001" ixy="0.0" ixz="0.0"
-                 iyy="0.001" iyz="0.0"
-                 izz="0.001" />
-      </inertial>
-    </link>
-    <joint name="caster_back_joint" type="fixed">
-      <parent link="base_link"/>
-      <child link="caster_back_link"/>
-      <origin xyz="-0.135 0.0 0.009" rpy="${-M_PI/2} 0 0"/>
-    </joint>
+    </collision>
+    <inertial>
+      <mass value="${caster_b_mass}" />
+      <origin xyz="0 0 0" />
+      <inertia ixx="0.001" ixy="0.0" ixz="0.0"
+               iyy="0.001" iyz="0.0"
+               izz="0.001" />
+    </inertial>
+  </link>
+  <joint name="caster_back_joint" type="fixed">
+    <parent link="base_link"/>
+    <child link="caster_back_link"/>
+    <origin xyz="-0.135 0.0 0.009" rpy="${-M_PI/2} 0 0"/>
+  </joint>
   <gazebo reference="caster_back_link">
     <turnGravityOff>false</turnGravityOff>
   </gazebo>
-<!-- Wheel Definitions -->
+  <!-- Wheel Definitions -->
   <wheel fb="front" lr="right" parent="base_link" translateX="0" translateY="0.5" flipY="1"/>
   <wheel fb="front" lr="left" parent="base_link" translateX="0" translateY="-0.5" flipY="1"/>
@@ -230,4 +230,5 @@
       <odometryTopic>odom</odometryTopic>
       <robotBaseFrame>base_footprint</robotBaseFrame>
+	  <legacyMode>true</legacyMode>
     </plugin>
   </gazebo>

File: chapter4_codes/ch4_seven_dof_arm_config/urdf/ch4_seven_dof_arm_gazebo.xacro (robot description, xacro)
@@ -130,5 +130,5 @@
     <axis xyz="-1 0 0" />
     <limit effort="300" velocity="1" lower="-2.61799387799" upper="1.98394848567"/>
-    <dynamics damping="50" friction="1"/>
+    <dynamics damping="0.1" friction="1"/>
   </joint>
   <!-- ///////////////////////////////////////////////////////////////////////////////////////////////////////////////////// -->
@@ -159,5 +159,5 @@
     <axis xyz="1 0 0" />
     <limit effort="300" velocity="1" lower="-1.19962513147" upper="1.89994105047" />
-    <dynamics damping="50" friction="1"/>
+    <dynamics damping="0.1" friction="1"/>
   </joint>
   <!-- ///////////////////////////////////////////////////////////////////////////////////////////////////////////////////// -->
@@ -189,5 +189,5 @@
     <axis xyz="-1 0 0" />
     <limit effort="300" velocity="1" lower="-2.61799387799" upper="0.705631162427" />
-    <dynamics damping="50" friction="1"/>
+    <dynamics damping="0.1" friction="1"/>
   </joint>
   <!-- ///////////////////////////////////////////////////////////////////////////////////////////////////////////////////// -->
@@ -218,5 +218,5 @@
     <axis xyz="1 0 0" />
     <limit effort="300" velocity="1" lower="-1.5953400194" upper="1.93281579274" />
-    <dynamics damping="50" friction="1"/>
+    <dynamics damping="0.1" friction="1"/>
   </joint>
   <!-- ///////////////////////////////////////////////////////////////////////////////////////////////////////////////////// -->
@@ -247,5 +247,5 @@
     <axis xyz="1 0 0" />
     <limit effort="300" velocity="1" lower="-2.61799387799" upper="2.6128806087" />
-    <dynamics damping="50" friction="1"/>
+    <dynamics damping="0.1" friction="1"/>
   </joint>
   <!-- WRIST ROLL LINK -->
@@ -275,5 +275,5 @@
     <axis xyz="1 0 0" />
     <limit effort="300" velocity="1" lower="-1.5953400194" upper="1.98394848567" />
-    <dynamics damping="50" friction="1"/>
+    <dynamics damping="0.1" friction="1"/>
   </joint>
   <!-- ///////////////////////////////////////////////////////////////////////////////////////////////////////////////////// -->
@@ -304,5 +304,5 @@
     <axis xyz="1 0 0" />
     <limit effort="300" velocity="1" lower="-2.61799387799" upper="2.6128806087" />
-    <dynamics damping="50" friction="1"/>
+    <dynamics damping="0.1" friction="1"/>
   </joint>
   <!-- ///////////////////////////////////////////////////////////////////////////////////////////////////////////////////// -->
@@ -337,5 +337,5 @@
                        soft_lower_limit="${-0.15 }"
                        soft_upper_limit="${ 0.0 }"/>
-    <dynamics damping="50" friction="1"/>
+    <dynamics damping="0.1" friction="1"/>
   </joint>
   <!-- ///////////////////////////////////////////////////////////////////////////////////////////////////////////////////// -->
@@ -362,5 +362,5 @@
     <limit effort="1" lower="-0.03" upper="0" velocity="1.0"/>
 	<!--    <mimic joint="gripper_finger_joint" multiplier="-1.0" offset="0.0" /> -->
-    <dynamics damping="50" friction="1"/>
+    <dynamics damping="0.1" friction="1"/>
   </joint>
   <!-- ///////////////////////////////////////////////////////////////////////////////////////////////////////////////////// -->
